Commit message: Completed physical object detection to virtual object identification pipeline. Additional filtering and  tweaks may be required.

File: cori_ws/install/cori_description/share/cori_description/urdf/cori.urdf.xacro (robot description, xacro)
@@ -41,5 +41,5 @@
     <parent link="base_link"/>
     <child link="torso"/>
-    <origin xyz="0 0 0.15" rpy="0 0 0"/>
+    <origin xyz="0 0 0" rpy="0 0 0"/>
   </joint>
   <link name="head">
@@ -66,5 +66,5 @@
     <child link="head"/>
     <origin xyz="0 0 0.0" rpy="0 0 0"/>
-    <axis xyz="0 0 1"/>  <!-- Fixed: inverted Z axis for correct direction -->
+    <axis xyz="0 0 1"/>
     <limit lower="-1.8" upper="1.8" effort="80" velocity="2.5"/>
     <dynamics damping="1.8" friction="0.9"/>
@@ -92,5 +92,5 @@
     <parent link="torso"/>
     <child link="pelvis"/>
-    <origin xyz="0 0 0" rpy="0 0 0"/>  <!-- Keep your spacing -->
+    <origin xyz="0 0 0" rpy="0 0 0"/>
   </joint>
   <link name="left_upper_arm">
@@ -116,6 +116,6 @@
     <parent link="torso"/>
     <child link="left_upper_arm"/>
-    <origin xyz="-0.07 0 0" rpy="0 0.15 0"/>  <!-- Keep your exact spacing -->
-    <axis xyz="1 0 0"/>  <!-- Shoulder rotation -->
+    <origin xyz="-0.07 0 0" rpy="0 0.15 0"/>
+    <axis xyz="1 0 0"/>
     <limit lower="-2.0" upper="2.0" effort="50" velocity="2.0"/>
     <dynamics damping="1.0" friction="0.5"/>
@@ -143,6 +143,6 @@
     <parent link="left_upper_arm"/>
     <child link="left_forearm"/>
-    <origin xyz="0 0 0" rpy="0 0 0"/>  <!-- Keep your exact spacing -->
-    <axis xyz="0 1 0"/>  <!-- Elbow bend -->
+    <origin xyz="0 0 0" rpy="0 0 0"/>
+    <axis xyz="0 1 0"/>
     <limit lower="-1.5" upper="1.5" effort="30" velocity="2.0"/>
     <dynamics damping="0.8" friction="0.3"/>
@@ -170,6 +170,6 @@
     <parent link="left_forearm"/>
     <child link="left_hand"/>
-    <origin xyz="0 0 0" rpy="0 0 0"/>  <!-- Keep your exact spacing -->
-    <axis xyz="0 0 1"/>  <!-- Wrist rotation -->
+    <origin xyz="0 0 0" rpy="0 0 0"/>
+    <axis xyz="0 0 1"/>
     <limit lower="-1.0" upper="1.0" effort="20" velocity="2.0"/>
     <dynamics damping="0.5" friction="0.2"/>
@@ -197,6 +197,6 @@
     <parent link="torso"/>
     <child link="right_upper_arm"/>
-    <origin xyz="0.07 0 0" rpy="0 -0.15 0"/>  <!-- Keep your exact spacing -->
-    <axis xyz="1 0 0"/>  <!-- Shoulder rotation -->
+    <origin xyz="0.07 0 0" rpy="0 -0.15 0"/>
+    <axis xyz="1 0 0"/>
     <limit lower="-2.0" upper="2.0" effort="50" velocity="2.0"/>
     <dynamics damping="1.0" friction="0.5"/>
@@ -224,6 +224,6 @@
     <parent link="right_upper_arm"/>
     <child link="right_forearm"/>
-    <origin xyz="0 0 0" rpy="0 0 0"/>  <!-- Keep your exact spacing -->
-    <axis xyz="0 1 0"/>  <!-- Elbow bend -->
+    <origin xyz="0 0 0" rpy="0 0 0"/>
+    <axis xyz="0 1 0"/>
     <limit lower="-1.5" upper="1.5" effort="30" velocity="2.0"/>
     <dynamics damping="0.8" friction="0.3"/>
@@ -251,6 +251,6 @@
     <parent link="right_forearm"/>
     <child link="right_hand"/>
-    <origin xyz="0 0 0" rpy="0 0 0"/>  <!-- Keep your exact spacing -->
-    <axis xyz="0 0 1"/>  <!-- Wrist rotation -->
+    <origin xyz="0 0 0" rpy="0 0 0"/>
+    <axis xyz="0 0 1"/>
     <limit lower="-1.0" upper="1.0" effort="20" velocity="2.0"/>
     <dynamics damping="0.5" friction="0.2"/>
@@ -278,6 +278,6 @@
     <parent link="pelvis"/>
     <child link="left_thigh"/>
-    <origin xyz="0 0 0" rpy="0 0 0"/>  <!-- Keep your exact spacing -->
-    <axis xyz="1 0 0"/>  <!-- Hip forward/back -->
+    <origin xyz="0 0 0" rpy="0 0 0"/>
+    <axis xyz="1 0 0"/>
     <limit lower="-1.0" upper="1.0" effort="60" velocity="1.5"/>
     <dynamics damping="1.5" friction="0.7"/>
@@ -305,6 +305,6 @@
     <parent link="left_thigh"/>
     <child link="left_shin"/>
-    <origin xyz="0 0 0" rpy="0 0 0"/>  <!-- Keep your exact spacing -->
-    <axis xyz="0 1 0"/>  <!-- Knee bend -->
+    <origin xyz="0 0 0" rpy="0 0 0"/>
+    <axis xyz="0 1 0"/>
     <limit lower="-1.5" upper="0.1" effort="40" velocity="1.5"/>
     <dynamics damping="1.2" friction="0.6"/>
@@ -332,5 +332,5 @@
     <parent link="left_shin"/>
     <child link="left_knee"/>
-    <origin xyz="0 0 0" rpy="0 0 0"/>  <!-- Keep your exact spacing -->
+    <origin xyz="0 0 0" rpy="0 0 0"/>
   </joint>
   <link name="left_foot">
@@ -356,6 +356,6 @@
     <parent link="left_knee"/>
     <child link="left_foot"/>
-    <origin xyz="0 0 0" rpy="0 0 0"/>  <!-- Keep your exact spacing -->
-    <axis xyz="0 1 0"/>  <!-- Ankle up/down -->
+    <origin xyz="0 0 0" rpy="0 0 0"/>
+    <axis xyz="0 1 0"/>
     <limit lower="-0.5" upper="0.5" effort="25" velocity="1.5"/>
     <dynamics damping="0.8" friction="0.4"/>
@@ -383,6 +383,6 @@
     <parent link="pelvis"/>
     <child link="right_thigh"/>
-    <origin xyz="0 0 0" rpy="0 0 0"/>  <!-- Keep your exact spacing -->
-    <axis xyz="1 0 0"/>  <!-- Hip forward/back -->
+    <origin xyz="0 0 0" rpy="0 0 0"/>
+    <axis xyz="1 0 0"/>
     <limit lower="-1.0" upper="1.0" effort="60" velocity="1.5"/>
     <dynamics damping="1.5" friction="0.7"/>
@@ -410,6 +410,6 @@
     <parent link="right_thigh"/>
     <child link="right_shin"/>
-    <origin xyz="0 0 0" rpy="0 0 0"/>  <!-- Keep your exact spacing -->
-    <axis xyz="0 1 0"/>  <!-- Knee bend -->
+    <origin xyz="0 0 0" rpy="0 0 0"/>
+    <axis xyz="0 1 0"/>
     <limit lower="-1.5" upper="0.1" effort="40" velocity="1.5"/>
     <dynamics damping="1.2" friction="0.6"/>
@@ -437,5 +437,5 @@
     <parent link="right_shin"/>
     <child link="right_knee"/>
-    <origin xyz="0 0 0" rpy="0 0 0"/>  <!-- Keep your exact spacing -->
+    <origin xyz="0 0 0" rpy="0 0 0"/>
   </joint>
   <link name="right_foot">
@@ -461,6 +461,6 @@
     <parent link="right_knee"/>
     <child link="right_foot"/>
-    <origin xyz="0 0 0" rpy="0 0 0"/>  <!-- Keep your exact spacing -->
-    <axis xyz="0 1 0"/>  <!-- Ankle up/down -->
+    <origin xyz="0 0 0" rpy="0 0 0"/>
+    <axis xyz="0 1 0"/>
     <limit lower="-0.5" upper="0.5" effort="25" velocity="1.5"/>
     <dynamics damping="0.8" friction="0.4"/>
@@ -477,5 +477,4 @@
     <material>Gazebo/Blue</material>
   </gazebo>
-  <!-- Joint Controllers for ALL movable joints -->
   <gazebo>
     <plugin filename="ignition-gazebo-joint-position-controller-system" name="ignition::gazebo::systems::JointPositionController">
